File: h2cboard_rev2/h2cboard.kicad_sch (KiCad schematic)
At the start: 19 parts, among them J1 HDMI_A, J2 SJ1-3525NG, J3 SCART-M, SW1 0S102011MS2QN1, U1 NX3303X, U2 ATtiny1604-SS

Commit message: New PCB layout for rev.2
Parts:
- U1: footprint Package_DFN_QFN:QFN-32-1EP_5x5mm_P0.5mm_EP3.65x3.65mm_ThermalVias -> footprints:QFN-32-1EP_5x5mm_P0.5mm_EP3.1x3.1mm_ThermalVias
Changed lines of the file:
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@@
 			)
 		)
-		(property "Footprint" "Package_DFN_QFN:QFN-32-1EP_5x5mm_P0.5mm_EP3.65x3.65mm_ThermalVias"
+		(property "Footprint" "footprints:QFN-32-1EP_5x5mm_P0.5mm_EP3.1x3.1mm_ThermalVias"
 			(at 104.14 92.71 0)
 			(effects
